Commit message: Feat: Added camera optical link to URDF and finalized Nav2 lifecycle sync

File: urdf/robot.urdf (robot description, URDF)
Before this commit: robot box_bot, 6 links, 5 joints
Links:
- added link camera_link_optical
Joints:
- added joint camera_optical_joint: type fixed, parent camera_link, child camera_link_optical, origin xyz=0 0 0 rpy=-1.5708 0 -1.5708
- joint camera_joint: origin xyz=0.25 0 0.15 -> xyz=0.25 0 0.15 rpy=0 0 0
